Commit message: clear useless document

File: diff_tracked/diff_tracked_base/urdf/bunker.xacro (robot description, xacro)
@@ -4,5 +4,4 @@
      For more information, please see http://wiki.ros.org/sw_urdf_exporter -->
 <robot  name="bunker_description" xmlns:xacro="http://www.ros.org/wiki/xacro">
-  <!-- <xacro:include filename="$(find diff_tracked_base)/urdf/bunker.urdf"/> -->
   <xacro:include filename="$(find diff_tracked_base)/urdf/laser_link.xacro"/>
   <xacro:include filename="$(find diff_tracked_base)/urdf/laser_driver.xacro"/>
@@ -41,9 +40,12 @@
     <collision>
       <origin
-        xyz="0.53 -0.392 -0.358"
-        rpy="1.57 0 3.14" />
-      <geometry>
-        <mesh
-          filename="package://diff_tracked_base/meshes/BUNKER.STL" scale="0.001 0.001 0.001" />
+        xyz="0 0 -0.12"
+        rpy="0 0 0" />
+      <geometry>
+        <!-- The original BUNKER mesh includes the tracks down to z=-0.358 m.
+             Using it as the chassis collision keeps the driven wheels above
+             the ground.  A raised chassis collision lets the road wheels
+             carry the vehicle while preserving the mesh as the visual. -->
+        <box size="0.90 0.60 0.25" />
       </geometry>
     </collision>
@@ -91,5 +93,5 @@
   <joint
     name="wheel1_joint"
-    type="revolute">
+    type="continuous">
     <origin
       xyz="0.44403 0.3495 -0.12853"
@@ -102,8 +104,6 @@
       xyz="0 0 1" />
     <limit
-      lower="-180"
-      upper="180"
-      effort="0"
-      velocity="0" />
+      effort="30"
+      velocity="20" />
   </joint>
   <link
@@ -149,5 +149,5 @@
   <joint
     name="wheel1.1_jont"
-    type="revolute">
+    type="continuous">
     <origin
       xyz="0.37551 0.3495 -0.22305"
@@ -160,8 +160,6 @@
       xyz="0 0 1" />
     <limit
-      lower="-180"
-      upper="180"
-      effort="0"
-      velocity="0" />
+      effort="30"
+      velocity="20" />
   </joint>
   <link
@@ -207,5 +205,5 @@
   <joint
     name="wheel1.2_joint"
-    type="revolute">
+    type="continuous">
     <origin
       xyz="0.29039 0.3495 -0.28104"
@@ -218,8 +216,6 @@
       xyz="0 0 1" />
     <limit
-      lower="-180"
-      upper="180"
-      effort="0"
-      velocity="0" />
+      effort="30"
+      velocity="20" />
   </joint>
   <link
@@ -265,5 +261,5 @@
   <joint
     name="wheel1.3_joint"
-    type="revolute">
+    type="continuous">
     <origin
       xyz="0.29603 0.3495 -0.087"
@@ -276,8 +272,6 @@
       xyz="0 0 -1" />
     <limit
-      lower="-180"
-      upper="180"
-      effort="0"
-      velocity="0" />
+      effort="30"
+      velocity="20" />
   </joint>
   <link
@@ -323,5 +317,5 @@
   <joint
     name="wheel2_joint"
-    type="revolute">
+    type="continuous">
     <origin
       xyz="0.44403 -0.3495 -0.12853"
@@ -334,8 +328,6 @@
       xyz="0 0 -1" />
     <limit
-      lower="-180"
-      upper="180"
-      effort="0"
-      velocity="0" />
+      effort="30"
+      velocity="20" />
   </joint>
   <link
@@ -381,5 +373,5 @@
   <joint
     name="wheel2.1_joint"
-    type="revolute">
+    type="continuous">
     <origin
       xyz="0.37551 -0.3495 -0.22305"
@@ -392,8 +384,6 @@
       xyz="0 0 -1" />
     <limit
-      lower="-180"
-      upper="180"
-      effort="0"
-      velocity="0" />
+      effort="30"
+      velocity="20" />
   </joint>
   <link
@@ -439,5 +429,5 @@
   <joint
     name="wheel2.2_joint"
-    type="revolute">
+    type="continuous">
     <origin
       xyz="0.29039 -0.3495 -0.28104"
@@ -448,10 +438,8 @@
       link="wheel2.2_Link" />
     <axis
-      xyz="0 0 -1" />
-    <limit
-      lower="-180"
-      upper="180"
-      effort="0"
-      velocity="0" />
+      xyz="0 0 1" />
+    <limit
+      effort="30"
+      velocity="20" />
   </joint>
   <link
@@ -497,5 +485,5 @@
   <joint
     name="wheel2.3_joint"
-    type="revolute">
+    type="continuous">
     <origin
       xyz="0.29603 -0.3495 -0.087"
@@ -508,8 +496,6 @@
       xyz="0 0 1" />
     <limit
-      lower="-180"
-      upper="180"
-      effort="0"
-      velocity="0" />
+      effort="30"
+      velocity="20" />
   </joint>
   <link
@@ -555,5 +541,5 @@
   <joint
     name="wheel3_joint"
-    type="revolute">
+    type="continuous">
     <origin
       xyz="-0.38871 0.295 -0.19381"
@@ -566,8 +552,6 @@
       xyz="0 0 -1" />
     <limit
-      lower="-180"
-      upper="180"
-      effort="0"
-      velocity="0" />
+      effort="30"
+      velocity="20" />
   </joint>
   <link
@@ -613,5 +597,5 @@
   <joint
     name="wheel3.1_joint"
-    type="revolute">
+    type="continuous">
     <origin
       xyz="-0.23111 0.3495 -0.27671"
@@ -624,8 +608,6 @@
       xyz="0 0 1" />
     <limit
-      lower="-180"
-      upper="180"
-      effort="0"
-      velocity="0" />
+      effort="30"
+      velocity="20" />
   </joint>
   <link
@@ -671,5 +653,5 @@
   <joint
     name="wheel3.2_joint"
-    type="revolute">
+    type="continuous">
     <origin
       xyz="0.043885 0.3495 -0.27671"
@@ -682,8 +664,6 @@
       xyz="0 0 1" />
     <limit
-      lower="-180"
-      upper="180"
-      effort="0"
-      velocity="0" />
+      effort="30"
+      velocity="20" />
   </joint>
   <link
@@ -729,5 +709,5 @@
   <joint
     name="wheel3.3_joint"
-    type="revolute">
+    type="continuous">
     <origin
       xyz="-0.28597 0.3495 -0.087"
@@ -740,8 +720,6 @@
       xyz="0 0 -1" />
     <limit
-      lower="-180"
-      upper="180"
-      effort="0"
-      velocity="0" />
+      effort="30"
+      velocity="20" />
   </joint>
   <link
@@ -787,5 +765,5 @@
   <joint
     name="wheel4_joint"
-    type="revolute">
+    type="continuous">
     <origin
       xyz="-0.38871 -0.295 -0.19381"
@@ -798,8 +776,6 @@
       xyz="0 0 1" />
     <limit
-      lower="-180"
-      upper="180"
-      effort="0"
-      velocity="0" />
+      effort="30"
+      velocity="20" />
   </joint>
   <link
@@ -845,5 +821,5 @@
   <joint
     name="wheel4.1_joint"
-    type="revolute">
+    type="continuous">
     <origin
       xyz="-0.23111 -0.3495 -0.27671"
@@ -856,8 +832,6 @@
       xyz="0 0 -1" />
     <limit
-      lower="-180"
-      upper="180"
-      effort="0"
-      velocity="0" />
+      effort="30"
+      velocity="20" />
   </joint>
   <link
@@ -903,5 +877,5 @@
   <joint
     name="wheel4.2_joint"
-    type="revolute">
+    type="continuous">
     <origin
       xyz="0.043885 -0.3495 -0.27671"
@@ -914,8 +888,6 @@
       xyz="0 0 -1" />
     <limit
-      lower="-180"
-      upper="180"
-      effort="0"
-      velocity="0" />
+      effort="30"
+      velocity="20" />
   </joint>
   <link
@@ -961,5 +933,5 @@
   <joint
     name="wheel4.3_joint"
-    type="revolute">
+    type="continuous">
     <origin
       xyz="-0.28597 -0.3495 -0.087"
@@ -972,8 +944,6 @@
       xyz="0 0 1" />
     <limit
-      lower="-180"
-      upper="180"
-      effort="0"
-      velocity="0" />
+      effort="30"
+      velocity="20" />
   </joint>
   <!-- /////////////////////////////////   gazebo color   ////////////////////////////////////// -->
@@ -981,5 +951,5 @@
      <material>Gazebo/Gray</material>
   </gazebo>
-  <gazebo>
+  <!-- <gazebo>
     <plugin name="object_controller" filename="libgazebo_ros_planar_move.so">
       <commandTopic>cmd_vel</commandTopic>
@@ -989,4 +959,79 @@
       <robotBaseFrame>base_link</robotBaseFrame>
     </plugin>
+  </gazebo> -->
+  <!-- <gazebo>
+    <plugin name="object_controller" filename="libgazebo_ros_planar_move.so">
+      <commandTopic>cmd_vel</commandTopic>
+      <odometryTopic>odom</odometryTopic>
+      <odometryFrame>odom</odometryFrame>
+      <odometryRate>20.0</odometryRate>
+      <leftFrontJoint>wheel1_2_joint</leftFrontJoint>
+      <rightFrontJoint>wheel2_2_joint</rightFrontJoint>
+      <leftRearJoint>wheel3_1_joint</leftRearJoint>
+      <rightRearJoint>wheel4_1_joint</rightRearJoint>
+      <robotBaseFrame>base_link</robotBaseFrame>
+    </plugin>
+  </gazebo> -->
+  <gazebo>
+    <plugin name="gazebo_ros_diff_drive" filename="libgazebo_ros_diff_drive.so">
+      <legacyMode>false</legacyMode>
+      <updateRate>100.0</updateRate>
+      <leftJoint>wheel1.2_joint</leftJoint>
+      <rightJoint>wheel2.2_joint</rightJoint>
+      <wheelSeparation>0.699</wheelSeparation>
+      <wheelDiameter>0.102</wheelDiameter>
+      <wheelTorque>30.0</wheelTorque>
+      <wheelAcceleration>1.8</wheelAcceleration>
+      <commandTopic>cmd_vel</commandTopic>
+      <odometryTopic>odom</odometryTopic>
+      <odometryFrame>odom</odometryFrame>
+      <robotBaseFrame>base_link</robotBaseFrame>
+      <publishOdom>true</publishOdom>
+      <publishOdomTF>false</publishOdomTF>
+      <publishWheelTF>false</publishWheelTF>
+      <publishWheelJointState>false</publishWheelJointState>
+    </plugin>
   </gazebo>
+  <gazebo reference="wheel1.2_Link">
+    <mu1>1.0</mu1>
+    <mu2>1.0</mu2>
+    <kp>100000.0</kp>
+    <kd>1.0</kd>
+  </gazebo>
+  <gazebo reference="wheel2.2_Link">
+    <mu1>1.0</mu1>
+    <mu2>1.0</mu2>
+    <kp>100000.0</kp>
+    <kd>1.0</kd>
+  </gazebo>
+  <gazebo>
+  <plugin name="joint_state_publisher"
+          filename="libgazebo_ros_joint_state_publisher.so">
+    <updateRate>50</updateRate>
+    <jointName>
+      wheel1_joint,
+      wheel1.1_jont,
+      wheel1.2_joint,
+      wheel1.3_joint,
+      wheel2_joint,
+      wheel2.1_joint,
+      wheel2.2_joint,
+      wheel2.3_joint,
+      wheel3_joint,
+      wheel3.1_joint,
+      wheel3.2_joint,
+      wheel3.3_joint,
+      wheel4_joint,
+      wheel4.1_joint,
+      wheel4.2_joint,
+      wheel4.3_joint
+    </jointName>
+  </plugin>
+</gazebo>
+  <!-- <gazebo>
+    <plugin name="gazebo_ros_control" filename="libgazebo_ros_control.so">
+      <robotSimType>gazebo_ros_control/DefaultRobotHWSim</robotSimType>
+      <legacyModeNS>true</legacyModeNS>
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
File: diff_tracked/diff_tracked_base/urdf/imu_link.xacro (robot description, xacro)
@@ -1,6 +1,6 @@
 <?xml version="1.0"?>
 <robot name="tracked_imu" xmlns:xacro="http://www.ros.org/wiki/xacro">
-  <!-- Installation pose relative to base_link. Adjust these values to the
-       measured IMU extrinsics on the real robot. -->
+  <!-- Installation pose relative to lidar_link. The IMU is stacked directly
+       above the lidar, without overlap between their visual geometries. -->
   <xacro:property name="imu_size" value="0.05" />
   <xacro:property name="imu_x" value="0.0"/>
@@ -31,5 +31,5 @@
   </link>
   <joint name="imu_joint" type="fixed">
-    <parent link="base_link"/>
+    <parent link="lidar_link"/>
     <child link="imu_link"/>
     <origin xyz="${imu_x} ${imu_y} ${imu_z}" rpy="0 0 0"/>
