Commit message: update

File: diff_car/diff_car_base/urdf/diff_car_laser_3d.xacro (robot description, xacro)
@@ -1,8 +1,8 @@
-<robot name="diff_car_laser"
+<robot name="diff_car_laser_3d"
   xmlns:xacro="http://wiki.ros.org/xacro">
   <xacro:include filename="head.xacro" />
   <xacro:include filename="base.xacro" />
   <xacro:include filename="laser.xacro" />
-  <xacro:include filename="laser_driver.xacro" />
+  <xacro:include filename="laser_3d_driver.xacro" />
   <xacro:include filename="imu.xacro" />
   <xacro:include filename="imu_driver.xacro" />

File: diff_car/diff_car_base/urdf/laser_3d_driver.xacro (robot description, xacro)
@@ -1,3 +1,3 @@
-<robot name="laser_driver"
+<robot name="laser_3d_driver"
   xmlns:xacro="http://wiki.ros.org/xacro">
   <gazebo reference="laser">

File: diff_car/diff_car_base/urdf/move.xacro (robot description, xacro)
@@ -1,5 +1,5 @@
 <robot name="diff_move"
   xmlns:xacro="http://wiki.ros.org/xacro">
-  <xacro:macro name="joint_trans" params="joint_name">
+  <!-- <xacro:macro name="joint_trans" params="joint_name">
     <transmission name="${joint_name}_trans">
       <type>transmission_interface/SimpleTransmission</type>
@@ -14,5 +14,5 @@
   </xacro:macro>
   <xacro:joint_trans joint_name="left_wheel2base_link" />
-  <xacro:joint_trans joint_name="right_wheel2base_link" />
+  <xacro:joint_trans joint_name="right_wheel2base_link" /> -->
   <gazebo>
     <plugin name="differential_drive_controller" filename="libgazebo_ros_diff_drive.so">

File: diff_tracked/diff_tracked_base/urdf/bunker.xacro (robot description, xacro)
@@ -1,13 +1,5 @@
 <?xml version="1.0" encoding="utf-8"?>
-<!-- This URDF was automatically created by SolidWorks to URDF Exporter! Originally created by Stephen Brawner (brawner@gmail.com)
-     Commit Version: 1.6.0-1-g15f4949  Build Version: 1.6.7594.29634
-     For more information, please see http://wiki.ros.org/sw_urdf_exporter -->
-<robot  name="bunker_description" xmlns:xacro="http://www.ros.org/wiki/xacro">
-  <xacro:include filename="$(find diff_tracked_base)/urdf/laser_link.xacro"/>
-  <xacro:include filename="$(find diff_tracked_base)/urdf/laser_driver.xacro"/>
-  <xacro:include filename="$(find diff_tracked_base)/urdf/imu_link.xacro"/>
-  <xacro:include filename="$(find diff_tracked_base)/urdf/imu_driver.xacro"/>
-  <link
-    name="base_link">
+<robot name="bunker" xmlns:xacro="http://www.ros.org/wiki/xacro">
+  <link name="base_link">
      <inertial>
       <origin
@@ -39,7 +31,5 @@
     </visual>
     <collision>
-      <origin
-        xyz="0 0 -0.12"
-        rpy="0 0 0" />
+      <origin xyz="0 0 -0.12" rpy="0 0 0" />
       <geometry>
         <!-- The original BUNKER mesh includes the tracks down to z=-0.358 m.
@@ -51,6 +41,5 @@
     </collision>
   </link>
-  <link
-    name="wheel1_Link">
+  <link name="wheel1_Link">
     <inertial>
       <origin
@@ -91,7 +80,5 @@
     </collision>
   </link>
-  <joint
-    name="wheel1_joint"
-    type="continuous">
+  <joint name="wheel1_joint" type="continuous">
     <origin
       xyz="0.44403 0.3495 -0.12853"
@@ -107,6 +94,5 @@
       velocity="20" />
   </joint>
-  <link
-    name="wheel1.1_Link">
+  <link name="wheel1.1_Link">
     <inertial>
       <origin
@@ -147,7 +133,5 @@
     </collision>
   </link>
-  <joint
-    name="wheel1.1_jont"
-    type="continuous">
+  <joint name="wheel1.1_jont" type="continuous">
     <origin
       xyz="0.37551 0.3495 -0.22305"
@@ -163,6 +147,5 @@
       velocity="20" />
   </joint>
-  <link
-    name="wheel1.2_Link">
+  <link name="wheel1.2_Link">
     <inertial>
       <origin
@@ -203,7 +186,5 @@
     </collision>
   </link>
-  <joint
-    name="wheel1.2_joint"
-    type="continuous">
+  <joint name="wheel1.2_joint" type="continuous">
     <origin
       xyz="0.29039 0.3495 -0.28104"
@@ -219,6 +200,5 @@
       velocity="20" />
   </joint>
-  <link
-    name="wheel1.3_Link">
+  <link name="wheel1.3_Link">
     <inertial>
       <origin
@@ -259,7 +239,5 @@
     </collision>
   </link>
-  <joint
-    name="wheel1.3_joint"
-    type="continuous">
+  <joint name="wheel1.3_joint" type="continuous">
     <origin
       xyz="0.29603 0.3495 -0.087"
@@ -275,6 +253,5 @@
       velocity="20" />
   </joint>
-  <link
-    name="wheel2_Link">
+  <link name="wheel2_Link">
     <inertial>
       <origin
@@ -315,7 +292,5 @@
     </collision>
   </link>
-  <joint
-    name="wheel2_joint"
-    type="continuous">
+  <joint name="wheel2_joint" type="continuous">
     <origin
       xyz="0.44403 -0.3495 -0.12853"
@@ -331,6 +306,5 @@
       velocity="20" />
   </joint>
-  <link
-    name="wheel2.1_Link">
+  <link name="wheel2.1_Link">
     <inertial>
       <origin
@@ -371,7 +345,5 @@
     </collision>
   </link>
-  <joint
-    name="wheel2.1_joint"
-    type="continuous">
+  <joint name="wheel2.1_joint" type="continuous">
     <origin
       xyz="0.37551 -0.3495 -0.22305"
@@ -387,6 +359,5 @@
       velocity="20" />
   </joint>
-  <link
-    name="wheel2.2_Link">
+  <link name="wheel2.2_Link">
     <inertial>
       <origin
@@ -427,7 +398,5 @@
     </collision>
   </link>
-  <joint
-    name="wheel2.2_joint"
-    type="continuous">
+  <joint name="wheel2.2_joint" type="continuous">
     <origin
       xyz="0.29039 -0.3495 -0.28104"
@@ -443,6 +412,5 @@
       velocity="20" />
   </joint>
-  <link
-    name="wheel2.3_Link">
+  <link name="wheel2.3_Link">
     <inertial>
       <origin
@@ -483,7 +451,5 @@
     </collision>
   </link>
-  <joint
-    name="wheel2.3_joint"
-    type="continuous">
+  <joint name="wheel2.3_joint" type="continuous">
     <origin
       xyz="0.29603 -0.3495 -0.087"
@@ -499,6 +465,5 @@
       velocity="20" />
   </joint>
-  <link
-    name="wheel3_Link">
+  <link name="wheel3_Link">
     <inertial>
       <origin
@@ -539,7 +504,5 @@
     </collision>
   </link>
-  <joint
-    name="wheel3_joint"
-    type="continuous">
+  <joint name="wheel3_joint" type="continuous">
     <origin
       xyz="-0.38871 0.295 -0.19381"
@@ -555,6 +518,5 @@
       velocity="20" />
   </joint>
-  <link
-    name="wheel3.1_Link">
+  <link name="wheel3.1_Link">
     <inertial>
       <origin
@@ -595,7 +557,5 @@
     </collision>
   </link>
-  <joint
-    name="wheel3.1_joint"
-    type="continuous">
+  <joint name="wheel3.1_joint" type="continuous">
     <origin
       xyz="-0.23111 0.3495 -0.27671"
@@ -611,6 +571,5 @@
       velocity="20" />
   </joint>
-  <link
-    name="wheel3.2_Link">
+  <link name="wheel3.2_Link">
     <inertial>
       <origin
@@ -651,7 +610,5 @@
     </collision>
   </link>
-  <joint
-    name="wheel3.2_joint"
-    type="continuous">
+  <joint name="wheel3.2_joint" type="continuous">
     <origin
       xyz="0.043885 0.3495 -0.27671"
@@ -667,6 +624,5 @@
       velocity="20" />
   </joint>
-  <link
-    name="wheel3.3_Link">
+  <link name="wheel3.3_Link">
     <inertial>
       <origin
@@ -707,7 +663,5 @@
     </collision>
   </link>
-  <joint
-    name="wheel3.3_joint"
-    type="continuous">
+  <joint name="wheel3.3_joint" type="continuous">
     <origin
       xyz="-0.28597 0.3495 -0.087"
@@ -723,6 +677,5 @@
       velocity="20" />
   </joint>
-  <link
-    name="wheel4_Link">
+  <link name="wheel4_Link">
     <inertial>
       <origin
@@ -763,7 +716,5 @@
     </collision>
   </link>
-  <joint
-    name="wheel4_joint"
-    type="continuous">
+  <joint name="wheel4_joint" type="continuous">
     <origin
       xyz="-0.38871 -0.295 -0.19381"
@@ -779,6 +730,5 @@
       velocity="20" />
   </joint>
-  <link
-    name="wheel4.1_Link">
+  <link name="wheel4.1_Link">
     <inertial>
       <origin
@@ -819,7 +769,5 @@
     </collision>
   </link>
-  <joint
-    name="wheel4.1_joint"
-    type="continuous">
+  <joint name="wheel4.1_joint" type="continuous">
     <origin
       xyz="-0.23111 -0.3495 -0.27671"
@@ -835,6 +783,5 @@
       velocity="20" />
   </joint>
-  <link
-    name="wheel4.2_Link">
+  <link name="wheel4.2_Link">
     <inertial>
       <origin
@@ -875,7 +822,5 @@
     </collision>
   </link>
-  <joint
-    name="wheel4.2_joint"
-    type="continuous">
+  <joint name="wheel4.2_joint" type="continuous">
     <origin
       xyz="0.043885 -0.3495 -0.27671"
@@ -891,6 +836,5 @@
       velocity="20" />
   </joint>
-  <link
-    name="wheel4.3_Link">
+  <link name="wheel4.3_Link">
     <inertial>
       <origin
@@ -931,7 +875,5 @@
     </collision>
   </link>
-  <joint
-    name="wheel4.3_joint"
-    type="continuous">
+  <joint name="wheel4.3_joint" type="continuous">
     <origin
       xyz="-0.28597 -0.3495 -0.087"
@@ -947,49 +889,6 @@
       velocity="20" />
   </joint>
-  <!-- /////////////////////////////////   gazebo color   ////////////////////////////////////// -->
- <gazebo reference="base_link">
+  <gazebo reference="base_link">
      <material>Gazebo/Gray</material>
-  </gazebo>
-  <!-- <gazebo>
-    <plugin name="object_controller" filename="libgazebo_ros_planar_move.so">
-      <commandTopic>cmd_vel</commandTopic>
-      <odometryTopic>odom</odometryTopic>
-      <odometryFrame>odom</odometryFrame>
-      <odometryRate>20.0</odometryRate>
-      <robotBaseFrame>base_link</robotBaseFrame>
-    </plugin>
-  </gazebo> -->
-  <!-- <gazebo>
-    <plugin name="object_controller" filename="libgazebo_ros_planar_move.so">
-      <commandTopic>cmd_vel</commandTopic>
-      <odometryTopic>odom</odometryTopic>
-      <odometryFrame>odom</odometryFrame>
-      <odometryRate>20.0</odometryRate>
-      <leftFrontJoint>wheel1_2_joint</leftFrontJoint>
-      <rightFrontJoint>wheel2_2_joint</rightFrontJoint>
-      <leftRearJoint>wheel3_1_joint</leftRearJoint>
-      <rightRearJoint>wheel4_1_joint</rightRearJoint>
-      <robotBaseFrame>base_link</robotBaseFrame>
-    </plugin>
-  </gazebo> -->
-  <gazebo>
-    <plugin name="gazebo_ros_diff_drive" filename="libgazebo_ros_diff_drive.so">
-      <legacyMode>false</legacyMode>
-      <updateRate>100.0</updateRate>
-      <leftJoint>wheel1.2_joint</leftJoint>
-      <rightJoint>wheel2.2_joint</rightJoint>
-      <wheelSeparation>0.699</wheelSeparation>
-      <wheelDiameter>0.102</wheelDiameter>
-      <wheelTorque>30.0</wheelTorque>
-      <wheelAcceleration>1.8</wheelAcceleration>
-      <commandTopic>cmd_vel</commandTopic>
-      <odometryTopic>odom</odometryTopic>
-      <odometryFrame>odom</odometryFrame>
-      <robotBaseFrame>base_link</robotBaseFrame>
-      <publishOdom>true</publishOdom>
-      <publishOdomTF>false</publishOdomTF>
-      <publishWheelTF>false</publishWheelTF>
-      <publishWheelJointState>false</publishWheelJointState>
-    </plugin>
   </gazebo>
   <gazebo reference="wheel1.2_Link">
@@ -1005,33 +904,3 @@
     <kd>1.0</kd>
   </gazebo>
-  <gazebo>
-  <plugin name="joint_state_publisher"
-          filename="libgazebo_ros_joint_state_publisher.so">
-    <updateRate>50</updateRate>
-    <jointName>
-      wheel1_joint,
-      wheel1.1_jont,
-      wheel1.2_joint,
-      wheel1.3_joint,
-      wheel2_joint,
-      wheel2.1_joint,
-      wheel2.2_joint,
-      wheel2.3_joint,
-      wheel3_joint,
-      wheel3.1_joint,
-      wheel3.2_joint,
-      wheel3.3_joint,
-      wheel4_joint,
-      wheel4.1_joint,
-      wheel4.2_joint,
-      wheel4.3_joint
-    </jointName>
-  </plugin>
-</gazebo>
-  <!-- <gazebo>
-    <plugin name="gazebo_ros_control" filename="libgazebo_ros_control.so">
-      <robotSimType>gazebo_ros_control/DefaultRobotHWSim</robotSimType>
-      <legacyModeNS>true</legacyModeNS>
-    </plugin>
-  </gazebo> -->
 </robot>

File: diff_tracked/diff_tracked_base/urdf/imu.xacro (robot description, xacro)
@@ -1,5 +1,5 @@
 <?xml version="1.0"?>
 <robot name="tracked_imu" xmlns:xacro="http://www.ros.org/wiki/xacro">
-  <!-- Installation pose relative to lidar_link. The IMU is stacked directly
+  <!-- Installation pose relative to laser. The IMU is stacked directly
        above the lidar, without overlap between their visual geometries. -->
   <xacro:property name="imu_size" value="0.05" />
@@ -7,5 +7,5 @@
   <xacro:property name="imu_y" value="0.0"/>
   <xacro:property name="imu_z" value="${laser_length / 2 + imu_size / 2}"/>
-  <link name="imu_link">
+  <link name="imu">
     <inertial>
       <mass value="0.05"/>
@@ -31,9 +31,9 @@
   </link>
   <joint name="imu_joint" type="fixed">
-    <parent link="lidar_link"/>
-    <child link="imu_link"/>
+    <parent link="laser"/>
+    <child link="imu"/>
     <origin xyz="${imu_x} ${imu_y} ${imu_z}" rpy="0 0 0"/>
   </joint>
-  <gazebo reference="imu_link">
+  <gazebo reference="imu">
     <material>Gazebo/Red</material>
   </gazebo>

File: diff_tracked/diff_tracked_base/urdf/laser.xacro (robot description, xacro)
@@ -1,12 +1,12 @@
 <?xml version="1.0"?>
-<robot name="tracked_lidar" xmlns:xacro="http://www.ros.org/wiki/xacro">
+<robot name="tracked_laser" xmlns:xacro="http://www.ros.org/wiki/xacro">
   <!-- Installation pose relative to base_link. Adjust these values to the
        measured lidar extrinsics on the real robot. -->
   <xacro:property name="laser_length" value="0.05" />
   <xacro:property name="laser_radius" value="0.05" />
-  <xacro:property name="lidar_x" value="0.0"/>
-  <xacro:property name="lidar_y" value="0.0"/>
-  <xacro:property name="lidar_z" value="${laser_length / 2}"/>
-  <link name="lidar_link">
+  <xacro:property name="laser_x" value="0.0"/>
+  <xacro:property name="laser_y" value="0.0"/>
+  <xacro:property name="laser_z" value="${laser_length / 2}"/>
+  <link name="laser">
     <inertial>
       <mass value="0.2"/>
@@ -33,8 +33,8 @@
   <joint name="lidar_joint" type="fixed">
     <parent link="base_link"/>
-    <child link="lidar_link"/>
-    <origin xyz="${lidar_x} ${lidar_y} ${lidar_z}" rpy="0 0 0"/>
+    <child link="laser"/>
+    <origin xyz="${laser_x} ${laser_y} ${laser_z}" rpy="0 0 0"/>
   </joint>
-  <gazebo reference="lidar_link">
+  <gazebo reference="laser">
     <material>Gazebo/Black</material>
   </gazebo>
