Commit message: update urdf and launch

File: diff_car/diff_car_base/urdf/move.xacro (robot description, xacro)
@@ -25,5 +25,5 @@
       <wheelAcceleration>1.8</wheelAcceleration>
       <commandTopic>/cmd_vel</commandTopic>
-      <odometryFrame>gz_odom</odometryFrame>
+      <odometryFrame>world</odometryFrame>
       <odometryTopic>/gz_odom</odometryTopic>
       <robotBaseFrame>base_footprint</robotBaseFrame>

File: diff_tracked/diff_tracked_base/urdf/bunker_laser_3d.xacro (robot description, xacro)
@@ -6,4 +6,5 @@
   <xacro:include filename="imu.xacro" />
   <xacro:include filename="imu_driver.xacro" />
+  <xacro:include filename="imu_pose_gt.xacro" />
   <xacro:include filename="move.xacro" />
 </robot>

File: diff_tracked/diff_tracked_base/urdf/imu_driver.xacro (robot description, xacro)
@@ -1,5 +1,5 @@
 <?xml version="1.0"?>
 <robot name="tracked_imu_driver" xmlns:xacro="http://www.ros.org/wiki/xacro">
-  <gazebo reference="imu_link">
+  <gazebo reference="imu">
     <sensor name="tracked_imu_sensor" type="imu">
       <always_on>true</always_on>
@@ -9,10 +9,10 @@
       <plugin name="tracked_imu_plugin" filename="libgazebo_ros_imu_sensor.so">
         <topicName>/imu</topicName>
-        <bodyName>imu_link</bodyName>
-        <updateRateHZ>300.0</updateRateHZ>
+        <bodyName>imu</bodyName>
+        <updateRateHZ>100.0</updateRateHZ>
         <gaussianNoise>0.0</gaussianNoise>
         <xyzOffset>0 0 0</xyzOffset>
         <rpyOffset>0 0 0</rpyOffset>
-        <frameName>imu_link</frameName>
+        <frameName>imu</frameName>
       </plugin>
     </sensor>

File: diff_tracked/diff_tracked_base/urdf/laser_3d_driver.xacro (robot description, xacro)
@@ -1,23 +1,23 @@
 <?xml version="1.0"?>
 <robot name="tracked_lidar_driver" xmlns:xacro="http://www.ros.org/wiki/xacro">
-  <gazebo reference="lidar_link">
+  <xacro:property name="PI" value="3.1415926"/>
+  <gazebo reference="laser">
     <sensor name="tracked_lidar_sensor" type="ray">
-      <always_on>true</always_on>
+      <pose>0 0 0 0 0 0</pose>
       <visualize>false</visualize>
       <update_rate>10</update_rate>
-      <pose>0 0 0 0 0 0</pose>
       <ray>
         <scan>
           <horizontal>
-            <samples>900</samples>
+            <samples>1800</samples>
             <resolution>1</resolution>
-            <min_angle>-${3.141592653589793}</min_angle>
-            <max_angle>${3.141592653589793}</max_angle>
+            <min_angle>-${PI}</min_angle>
+            <max_angle> ${PI}</max_angle>
           </horizontal>
           <vertical>
-            <samples>16</samples>
+            <samples>32</samples>
             <resolution>1</resolution>
-            <min_angle>-${15.0 * 3.141592653589793 / 180.0}</min_angle>
-            <max_angle>${15.0 * 3.141592653589793 / 180.0}</max_angle>
+            <min_angle>-${10.0*PI/180.0}</min_angle>
+            <max_angle> ${30.0*PI/180.0}</max_angle>
           </vertical>
         </scan>
@@ -30,13 +30,13 @@
           <type>gaussian</type>
           <mean>0.0</mean>
-          <stddev>0.008</stddev>
+          <stddev>0.0</stddev>
         </noise>
       </ray>
-      <plugin name="tracked_lidar_plugin" filename="libgazebo_ros_velodyne_laser.so">
+      <plugin name="gazebo_ros_laser_controller" filename="libgazebo_ros_velodyne_laser.so">
         <topicName>/scan</topicName>
-        <frameName>lidar_link</frameName>
+        <frameName>laser</frameName>
         <organize_cloud>false</organize_cloud>
-        <min_range>0.15</min_range>
-        <max_range>100.0</max_range>
+        <min_range>0.9</min_range>
+        <max_range>100</max_range>
         <gaussianNoise>0.008</gaussianNoise>
       </plugin>

File: diff_tracked/diff_tracked_base/urdf/move.xacro (robot description, xacro)
@@ -3,20 +3,24 @@
   <gazebo>
     <plugin name="differential_drive_controller" filename="libgazebo_ros_diff_drive.so">
-      <legacyMode>false</legacyMode>
       <updateRate>100.0</updateRate>
       <leftJoint>wheel1.2_joint</leftJoint>
       <rightJoint>wheel2.2_joint</rightJoint>
-      <wheelSeparation>0.60</wheelSeparation>
+      <wheelSeparation>0.6</wheelSeparation>
       <wheelDiameter>0.102</wheelDiameter>
-      <wheelTorque>30.0</wheelTorque>
+      <wheelTorque>30</wheelTorque>
       <wheelAcceleration>1.8</wheelAcceleration>
       <commandTopic>/cmd_vel</commandTopic>
+      <odometryFrame>world</odometryFrame>
       <odometryTopic>/gz_odom</odometryTopic>
-      <odometryFrame>gz_odom</odometryFrame>
       <robotBaseFrame>base_link</robotBaseFrame>
+      <!-- Set to true to swap right and left wheels, defaults to true -->
+      <legacyMode>false</legacyMode>
+      <!-- joint_state_publisher + robot_state_publisher own all wheel-link TFs.
+           Publishing these two here as well produces TF_REPEATED_DATA in RViz. -->
+      <publishWheelTF>false</publishWheelTF>
+      <!-- Set to true to publish sensor_msgs/JointState on /joint_states for the wheel joints, defaults to false -->
+      <publishWheelJointState>false</publishWheelJointState>
+      <!-- Set to true to publish transforms for the odometry, defaults to true -->
       <publishOdom>true</publishOdom>
-      <publishOdomTF>false</publishOdomTF>
-      <publishWheelTF>false</publishWheelTF>
-      <publishWheelJointState>false</publishWheelJointState>
     </plugin>
   </gazebo>
